File: LED-100.kicad_pcb (KiCad board)
At the start: 2 copper layers, 100 x 100 mm, 102 parts, among them J2 LDA100_2_J2, J3 LDA100_2_J3, J4 LDA100_2_J4, J5 xtra, J7 Conn_01x01, J8 Conn_01x08, SW1 SW_SPDT, U1 TLC5947DAP, U2 TLC5947DAP, U3 TLC5947DAP, U4 TEENSY 4.0

Commit message: WIP
Parts:
- removed D1, D10, D11, D12, D13, D14, D15, D16, D17, D18, D19, D2, D20, D21a1, D21b1, D22, D23a1, D23b1, D24, D25, D26, D27, D28, D29, D30, D31, D32, D33, D34, D35, D36, D37, D38, D39a1, D39b1, D3a1, D3b1, D4, D40a1, D40b1, D41, D42, D43, D44, D45, D46, D47, D48, D49, D5, D50, D51, D52a1, D52b1, D53a1, D53b1, D54, D55, D56, D57, D58, D59, D6, D60, D69, D70, D71, D72, D7a1, D7b1, D8, D9: LED_Small, LED_SMD:LED_0805_2012Metric_Pad1.15x1.40mm_HandSolder
- removed R5: 100k, Resistor_THT:R_Axial_DIN0204_L3.6mm_D1.6mm_P5.08mm_Horizontal
- removed SELECT: SW_SPST, Button_Switch_THT:SW_PUSH_6mm_H5mm
- removed SW1: SW_SPDT, MyParts:SWITCH_SPDT-SLW-12689-4A-N-D
- added SW2: SW_SPST, Button_Switch_THT:SW_PUSH_6mm_H5mm, F.Cu at (54.0, 145.0)
- J8: value Conn_01x08 -> Conn_01x07; footprint Connector_PinHeader_2.54mm:PinHeader_1x08_P2.54mm_Vertical -> Connector_PinHeader_2.54mm:PinHeader_1x07_P2.54mm_Vertical
- RV1: value R_Potentiometer_US -> 100k
- moved H2 197.4 mm to (22.0, 150.0)
- moved H3 174.5 mm to (258.0, 61.0)
- moved REF** 139.1 mm to (246.0, 147.5), turned to 180 degrees
- moved J1 115.8 mm to (260.0, 139.0), turned to 180 degrees
- moved JP1 104.9 mm to (64.0, 129.3)
- moved U1 104.5 mm to (248.7, 107.3), turned to 90 degrees
- moved R1 99.0 mm to (241.5, 101.5), turned to 90 degrees
- moved C1 94.3 mm to (241.5, 104.5), turned to -90 degrees
- moved TP1 87.0 mm to (30.5, 125.5)
- moved TP2 86.3 mm to (30.5, 135.0)
- moved R4 84.9 mm to (76.0, 127.5), turned to 180 degrees
- moved H1 83.2 mm to (22.0, 61.0)
- moved J4 82.8 mm to (20.0, 122.2)
- moved U4 78.3 mm to (50.4, 112.2), turned to 0 degrees
- moved J8 73.7 mm to (64.0, 107.3), turned to 0 degrees
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Connections:
- RV1 pad 1: +5V -> +3.3V
- U1 pad 29: MISO_B -> Net-(J7-Pin_1)
- U1 pad 4: MISO_A -> MISO_C
- U2 pad 29: MISO_C -> MISO_B
- U2 pad 4: MISO_B -> MISO_A
- U3 pad 29: Net-(J7-Pin_1) -> MISO_C
- U3 pad 4: MISO_C -> MISO_B
- U4 pad 11: FADESPEED -> unconnected-(U4-9-Pad11)
- U4 pad 18: Net-(J8-Pin_8) -> Net-(J8-Pin_7)
- U4 pad 19: Net-(J8-Pin_7) -> Net-(J8-Pin_6)
- U4 pad 20: Net-(J8-Pin_6) -> Net-(J8-Pin_5)
- U4 pad 21: Net-(J8-Pin_5) -> Net-(J8-Pin_4)
- U4 pad 22: Net-(J8-Pin_4) -> Net-(J8-Pin_3)
- U4 pad 23: Net-(J8-Pin_3) -> Net-(J8-Pin_2)
- U4 pad 24: Net-(J8-Pin_2) -> Net-(J8-Pin_1)
- U4 pad 25: Net-(J8-Pin_1) -> FADESPEED
- U4 pad 26: unconnected-(U4-3.3V-Pad26) -> +3.3V
Routing:
- net /TEST5V: track 263.5 -> 0.00 mm, vias 7 -> 0
- net BLANK: track 97.9 -> 222.8 mm, vias 3 -> 6
- net SCK: track 99.9 -> 224.5 mm, vias 4 -> 6
- net LAT: track 123.8 -> 245.2 mm, vias 5 -> 6
- net +5V: track 214.2 -> 319.4 mm, vias 4 -> 6
- net Net-(J4-AD3): track 10.7 -> 30.2 mm
- net MISO_B: track 71.7 -> 90.8 mm, vias 2 -> 0
- net MISO_C: track 38.7 -> 57.7 mm
- net Net-(J4-AD2): track 12.5 -> 30.2 mm
- net Net-(J4-AD1): track 14.1 -> 30.2 mm
- net +3.3V: track 0.00 -> 15.4 mm
- net Net-(J4-AD0): track 16.6 -> 30.2 mm
- net QX4: track 16.8 -> 29.9 mm, vias 1 -> 0
- net Net-(J4-Strobe): track 18.7 -> 30.2 mm
- net QX3: track 19.6 -> 30.7 mm, vias 1 -> 0
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Other:
- board size 100 x 100 mm -> 246 x 99 mm
- board text added: "Q20"
- board text added: "Rev. 4"
- board text added: "select"
- board text removed: "1"
- board text removed: "Blank Pullup"
- board text removed: "Debug LEDs"
- board text removed: "OFF"
- board text removed: "ON"
- board text removed: "Rev. 3"
