File: LED-100.kicad_pcb (KiCad board)
At the start: 2 copper layers, 246 x 99 mm, 28 parts, among them J2 LDA100_2_J2, J3 LDA100_2_J3, J4 LDA100_2_J4, J5 xtra, J7 Conn_01x01, J8 Conn_01x07, SW2 SW_SPST, U1 TLC5947DAP, U2 TLC5947DAP, U3 TLC5947DAP, U4 TEENSY 4.0

Commit message: Rev 5
Parts:
- removed JP1: SolderJumper_2_Bridged, Jumper:SolderJumper-2_P1.3mm_Bridged_Pad1.0x1.5mm
- removed REF**: OSHW-Logo2_7.3x6mm_SilkScreen, Symbol:OSHW-Logo2_7.3x6mm_SilkScreen
- added C4: .1u, Capacitor_THT:C_Disc_D3.0mm_W1.6mm_P2.50mm, F.Cu at (40.0, 116.4)
- added C5: .1u, Capacitor_THT:C_Disc_D3.0mm_W1.6mm_P2.50mm, F.Cu at (49.9, 106.9)
- added C6: 47u, Capacitor_THT:CP_Radial_D6.3mm_P2.50mm, F.Cu at (33.0, 80.5)
- added RN1: 1M, Resistor_THT:R_Array_SIP10, F.Cu at (33.0, 108.5)
- added RV2: 100k, Potentiometer_THT:Potentiometer_Bourns_PTV09A-1_Single_Vertical, F.Cu at (44.1, 130.1)
- added U5: ~, Package_SO:TSSOP-14_4.4x5mm_P0.65mm, F.Cu at (52.1, 99.6)
- added U6: ~, Package_SO:TSSOP-14_4.4x5mm_P0.65mm, F.Cu at (42.1, 109.6)
- C1, C2, C3: footprint Capacitor_THT:C_Disc_D3.0mm_W2.0mm_P2.50mm -> Capacitor_THT:C_Disc_D3.0mm_W1.6mm_P2.50mm
- J6: renamed from J8; value Conn_01x07 -> Conn_01x05; footprint Connector_PinHeader_2.54mm:PinHeader_1x07_P2.54mm_Vertical -> Connector_PinHeader_2.54mm:PinHeader_1x05_P2.54mm_Vertical
- RV1: footprint Potentiometer_THT:Potentiometer_Piher_PT-10-V10_Vertical -> Potentiometer_THT:Potentiometer_Bourns_PTV09A-1_Single_Vertical
- moved J7 196.8 mm to (45.0, 77.0)
- moved U1 182.5 mm to (69.1, 74.2), turned to 180 degrees
- moved R1 181.3 mm to (61.5, 79.5), turned to 180 degrees
- moved J1 178.7 mm to (100.7, 58.2), turned to -90 degrees
- moved C1 175.9 mm to (67.0, 82.5), turned to 180 degrees
- moved H3 147.0 mm to (111.0, 61.0)
- moved H4 147.0 mm to (111.0, 150.0)
- moved C2 130.6 mm to (81.5, 129.5)
- moved R3 128.1 mm to (93.0, 94.0), turned to 180 degrees
- moved U3 117.8 mm to (98.0, 101.0), turned to 90 degrees
- moved SW2 58.5 mm to (58.3, 86.6), turned to -45 degrees
- moved J3 58.0 mm to (113.6, 139.8), turned to 180 degrees
- moved J5 48.0 mm to (98.0, 133.2), turned to 0 degrees
- moved TP2 47.8 mm to (45.0, 89.5)
- moved TP1 44.4 mm to (45.0, 83.5)
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Connections:
- net MISO_B renamed MOSI_B
- net MISO_C renamed MOSI_C
- C1 pad 1: +5V -> +3.3V
- C2 pad 1: +5V -> +3.3V
- C3 pad 1: +5V -> +3.3V
- J5 pad 1: QX1 -> QX4
- J5 pad 2: QX2 -> QX3
- J5 pad 3: QX3 -> QX2
- J5 pad 4: QX4 -> QX1
- R4 pad 1: +5V -> +3.3V
- SW2 pad 1: GND -> SW_SELECT
- SW2 pad 2: SW_SELECT -> GND
- U1 pad 32: +5V -> +3.3V
- U2 pad 32: +5V -> +3.3V
- U2 pad 4: MISO_A -> MOSI_A
- U3 pad 32: +5V -> +3.3V
- U4 pad 10: Net-(J4-PD3) -> Net-(U4-8)
- U4 pad 11: unconnected-(U4-9-Pad11) -> Net-(U4-9)
- U4 pad 12: unconnected-(U4-10-Pad12) -> Net-(U4-10)
- U4 pad 13: SW_SELECT -> MOSI_A
- U4 pad 14: MISO_A -> unconnected-(U4-12_MISO-Pad14)
- U4 pad 18: Net-(J8-Pin_7) -> BRIGHTNESS
- U4 pad 19: Net-(J8-Pin_6) -> FADESPEED
- U4 pad 2: Net-(J4-AD3) -> unconnected-(U4-0-Pad2)
- U4 pad 25: FADESPEED -> SW_SELECT
- U4 pad 3: Net-(J4-AD2) -> unconnected-(U4-1-Pad3)
- U4 pad 4: Net-(J4-AD1) -> Net-(U4-2)
- U4 pad 5: Net-(J4-AD0) -> Net-(U4-3)
- U4 pad 6: Net-(J4-Strobe) -> Net-(U4-4)
- U4 pad 7: Net-(J4-PD0) -> Net-(U4-5)
- U4 pad 8: Net-(J4-PD1) -> Net-(U4-6)
- U4 pad 9: Net-(J4-PD2) -> Net-(U4-7)
Routing:
- net +5V: track 319.4 -> 104.0 mm, vias 6 -> 0
- net +3.3V: track 15.4 -> 164.3 mm, vias 0 -> 2
- net BLANK: track 222.8 -> 101.1 mm, vias 6 -> 5
- net LAT: track 245.2 -> 126.9 mm, vias 6 -> 4
- net SCK: track 224.5 -> 113.1 mm, vias 6 -> 5
- net MISO_A: track 67.7 -> 0.00 mm
- net MOSI_B: track 90.8 -> 42.1 mm
- net MOSI_A: track 0.00 -> 40.2 mm, vias 0 -> 1
- net MOSI_C: track 57.7 -> 33.5 mm
- net Net-(J4-AD3): track 30.2 -> 50.3 mm
- net BRIGHTNESS: track 0.00 -> 18.7 mm
- net Net-(J4-AD2): track 30.2 -> 47.0 mm
- net GND: track 0.00 -> 16.0 mm, vias 0 -> 2
- net QX3: track 30.7 -> 17.0 mm
- net QX1: track 32.2 -> 18.6 mm
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Other:
- board size 246 x 99 mm -> 99 x 99 mm
- board text added: "QX1"
- board text added: "QX2"
- board text added: "QX3"
- board text added: "QX4"
- board text added: "Rev. 5"
- board text added: "boop"
- board text added: "bright"
- board text removed: "BLANK"
- board text removed: "Curr. Set"
- board text removed: "LATCH"
- board text removed: "MISO"
- board text removed: "Rev. 4"
- board text removed: "SCK"
- board text removed: "SOut"
- board text removed: "select"
